File: UccMicroDuino/UccMicroDuino.kicad_pcb (KiCad board)
At the start: 2 copper layers, 8 parts, among them J1 Conn_01x10_Socket, J2 USB_A, U1 ATtiny85-20S

Commit message: Add files via upload
Parts:
- added D3: D_Zener, Diode_SMD:D_SOD-123, F.Cu at (210.7, 77.0)
- added D4: LED, ledSmd:ledSMD, F.Cu at (184.8, 88.0)
- added R2: R, Resistor_SMD:R_0805_2012Metric_Pad1.20x1.40mm_HandSolder, F.Cu at (193.0, 78.0)
- added R3: R, Resistor_SMD:R_0805_2012Metric_Pad1.20x1.40mm_HandSolder, F.Cu at (202.0, 79.0)
- added R4: R, Resistor_SMD:R_0805_2012Metric_Pad1.20x1.40mm_HandSolder, F.Cu at (178.0, 89.0)
- added R5: R, Resistor_SMD:R_0805_2012Metric_Pad1.20x1.40mm_HandSolder, F.Cu at (173.0, 89.0)
- U1: footprint Package_SO:SOIC-8W_5.3x5.3mm_P1.27mm -> Package_SO:SOIC-8_5.3x5.3mm_P1.27mm
- moved D2 75.8 mm to (203.0, 72.7), turned to 90 degrees
- moved J1 67.0 mm to (182.9, 100.0), turned to 90 degrees
- moved U1 62.8 mm to (193.6, 92.9), turned to 180 degrees
- moved C1 48.3 mm to (174.0, 100.0), turned to -90 degrees
- moved D1 46.1 mm to (174.8, 78.0), turned to 180 degrees
- moved J2 44.6 mm to (176.0, 65.0), turned to -90 degrees
- moved D5 39.4 mm to (175.0, 84.0)
- moved R1 38.6 mm to (177.0, 74.0), turned to 90 degrees
- renumbered D3 to D5
Connections:
- C1 pad 1: unconnected-(C1-Pad1) -> +5V
- C1 pad 2: unconnected-(C1-Pad2) -> GND
- D1 pad 2: unconnected-(D1-A-Pad2) -> Net-(D1-A)
- D2 pad 1: unconnected-(D2-K-Pad1) -> Net-(D2-K)
- D2 pad 2: unconnected-(D2-A-Pad2) -> GND
- D5 pad 1: unconnected-(D3-K-Pad1) -> Net-(D5-K)
- D5 pad 2: unconnected-(D3-A-Pad2) -> +5V
- J1 pad 1: unconnected-(J1-Pin_1-Pad1) -> +5V
- J1 pad 2: unconnected-(J1-Pin_2-Pad2) -> GND
- J1 pad 4: unconnected-(J1-Pin_4-Pad4) -> Net-(J1-Pin_4)
- J1 pad 5: unconnected-(J1-Pin_5-Pad5) -> Net-(D4-A)
- J1 pad 6: unconnected-(J1-Pin_6-Pad6) -> Net-(J1-Pin_6)
- J1 pad 7: unconnected-(J1-Pin_7-Pad7) -> Net-(J1-Pin_7)
- J1 pad 8: unconnected-(J1-Pin_8-Pad8) -> Net-(J1-Pin_8)
- J1 pad 9: unconnected-(J1-Pin_9-Pad9) -> Net-(J1-Pin_9)
- J2 pad 1: unconnected-(J2-VBUS-Pad1) -> Net-(D1-A)
- J2 pad 2: unconnected-(J2-D--Pad2) -> Net-(D2-K)
- J2 pad 3: unconnected-(J2-D+-Pad3) -> Net-(D3-K)
- J2 pad 4: unconnected-(J2-GND-Pad4) -> GND
- R1 pad 2: unconnected-(R1-Pad2) -> Net-(D2-K)
- U1 pad 1: unconnected-(U1-~{RESET}/PB5-Pad1) -> Net-(J1-Pin_9)
- U1 pad 2: unconnected-(U1-XTAL1/PB3-Pad2) -> Net-(J1-Pin_7)
- U1 pad 3: unconnected-(U1-XTAL2/PB4-Pad3) -> Net-(J1-Pin_8)
- U1 pad 4: unconnected-(U1-GND-Pad4) -> GND
- U1 pad 5: unconnected-(U1-AREF/PB0-Pad5) -> Net-(J1-Pin_4)
- U1 pad 6: unconnected-(U1-PB1-Pad6) -> Net-(D4-A)
- U1 pad 7: unconnected-(U1-PB2-Pad7) -> Net-(J1-Pin_6)
- U1 pad 8: unconnected-(U1-VCC-Pad8) -> +5V
Routing:
- net GND: track 0.00 -> 149.0 mm
- net +5V: track 0.00 -> 65.0 mm
- net Net-(D3-K): track 0.00 -> 48.6 mm
- net Net-(J1-Pin_8): track 0.00 -> 38.2 mm
- net Net-(D2-K): track 0.00 -> 37.3 mm
- net Net-(J1-Pin_7): track 0.00 -> 25.3 mm
- net Net-(D4-A): track 0.00 -> 23.2 mm
- net Net-(D1-A): track 0.00 -> 13.4 mm
- net Net-(J1-Pin_4): track 0.00 -> 12.9 mm
- net Net-(J1-Pin_6): track 0.00 -> 12.3 mm
- net Net-(J1-Pin_9): track 0.00 -> 8.21 mm
- net Net-(D4-K): track 0.00 -> 5.00 mm
- net Net-(D5-K): track 0.00 -> 4.08 mm
Other:
- board outline added: 45 x 45 mm
