File: UccMicroDuino/UccMicroDuino.kicad_sch (KiCad schematic)
At the start: 8 parts, among them J2 Conn_01x10_Socket, J2 USB_A, U2 ATtiny85-20S

Commit message: Add files via upload
Parts:
- added D3: D_Zener, Diode_SMD:D_SOD-123, symbol Device:D_Zener
- added D4: LED, ledSmd:ledSMD, symbol Device:LED
- added R2, R3, R4, R5: R, Resistor_SMD:R_0805_2012Metric_Pad1.20x1.40mm_HandSolder, symbol Device:R
- U1: renamed from U2; footprint Package_SO:SOIC-8W_5.3x5.3mm_P1.27mm -> Package_SO:SOIC-8_5.3x5.3mm_P1.27mm
- renumbered D5 to D1, D1 to D2, D3 to D5, J2 to J1
Connections:
- net +5V: now also C1.1, D5.2 (A), J1.1 (Pin_1), U1.8 (VCC)
- net GND: now also C1.2, D2.2 (A), J1.2 (Pin_2), J2.4 (GND), U1.4 (GND), D3.2 (A), R4.2, R5.1
- net at D5.1 (K): now also R5.2
- net at R1.2: now also D2.1 (K), J2.2 (D-), R2.1
- net at U1.1 (~{RESET}/PB5): now also J1.9 (Pin_9)
- net at U1.2 (XTAL1/PB3): now also J1.7 (Pin_7), R2.2
- net at U1.3 (XTAL2/PB4): now also J1.8 (Pin_8), R3.2
- net at U1.5 (AREF/PB0): now also J1.4 (Pin_4)
- net at U1.6 (PB1): now also J1.5 (Pin_5), D4.2 (A)
- net at U1.7 (PB2): now also J1.6 (Pin_6)
- net at J2.1 (VBUS): now also D1.2 (A)
- net at J2.3 (D+): now also D3.1 (K), R3.1
- new net: D4.1 (K), R4.1
- no-connect marks 0 -> 2
Other:
- moved on the sheet: D2, D5, U1
